Commit message: Add Lidar

File: catkin_ws/src/my_robot/urdf/my_robot.xacro (robot description, xacro)
@@ -29,4 +29,5 @@
         <box size=".4 .2 .1"/>
       </geometry>
+         <material name="blue"/>
     </visual>
     <collision name='back_caster_collision'>
@@ -76,4 +77,5 @@
         <cylinder radius="0.1" length="0.05"/>
       </geometry>
+         <material name="Green"/>
     </visual>
 </link>
@@ -107,4 +109,5 @@
         <cylinder radius="0.1" length="0.05"/>
       </geometry>
+         <material name="Green"/>
     </visual>
 </link>
@@ -138,4 +141,5 @@
         <box size="0.05 0.05 0.05"/>
       </geometry>
+         <material name="Red"/>
     </visual>
 </link>
@@ -146,3 +150,32 @@
     <axis xyz="0 1 0" rpy="0 0 0"/>
 </joint>
+<link name='hokuyo'>
+    <inertial>
+      <mass value="1e-5"/>
+      <origin xyz="0 0 0" rpy=" 0 0 0"/>
+      <inertia
+          ixx="1e-6" ixy="0" ixz="0"
+          iyy="1e-6" iyz="0"
+          izz="1e-6"
+      />
+    </inertial>
+    <collision name='collision'>
+      <origin xyz="0 0 0" rpy=" 0 0 0"/>
+      <geometry>
+        <box size="0.1 0.1 0.1"/>
+      </geometry>
+    </collision>
+    <visual name='visual'>
+      <origin xyz="0 0 0" rpy=" 0 0 0"/>
+      <geometry>
+	    <mesh filename="package://my_robot/meshes/hokuyo.dae" />
+      </geometry>
+    </visual>
+</link>
+<joint type="fixed" name="hokuyo_joint">
+    <origin xyz="0.15 0 .1" rpy="0 0 0"/>
+    <child link="hokuyo"/>
+    <parent link="chassis"/>
+    <axis xyz="0 1 0" rpy="0 0 0"/>
+</joint>
 </robot>

Commit message: Added Camera, Lidar, and Diff. Drive Controller plugins to Gazebo for publishing data/receiving commands

File: catkin_ws/src/my_robot/urdf/my_robot.xacro (robot description, xacro)
@@ -1,4 +1,5 @@
 <?xml version='1.0'?>
 <robot name="my_robot" xmlns:xacro="http://www.ros.org/wiki/xacro">
+  <xacro:include filename="$(find my_robot)/urdf/my_robot.gazebo" />
   <link name="robot_footprint"></link>
   <joint name="robot_footprint_joint" type="fixed">
@@ -29,5 +30,5 @@
         <box size=".4 .2 .1"/>
       </geometry>
-         <material name="blue"/>
+         <material name="Gazebo/Blue"/>
     </visual>
     <collision name='back_caster_collision'>

Commit message: Add RViz; try to set colors

File: catkin_ws/src/my_robot/urdf/my_robot.xacro (robot description, xacro)
@@ -30,5 +30,5 @@
         <box size=".4 .2 .1"/>
       </geometry>
-         <material name="Gazebo/Blue"/>
+         <material name="green"/>
     </visual>
     <collision name='back_caster_collision'>
@@ -78,5 +78,5 @@
         <cylinder radius="0.1" length="0.05"/>
       </geometry>
-         <material name="Green"/>
+         <material name="green"/>
     </visual>
 </link>
@@ -110,5 +110,5 @@
         <cylinder radius="0.1" length="0.05"/>
       </geometry>
-         <material name="Green"/>
+         <material name="green"/>
     </visual>
 </link>
@@ -142,5 +142,5 @@
         <box size="0.05 0.05 0.05"/>
       </geometry>
-         <material name="Red"/>
+         <material name="red"/>
     </visual>
 </link>

Commit message: Change dimensions of robot; fix duplicate my_robot error message; update process_image.cpp to handle correct format (RGB)

File: catkin_ws/src/my_robot/urdf/my_robot.xacro (robot description, xacro)
@@ -22,5 +22,5 @@
       <origin xyz="0 0 0" rpy=" 0 0 0"/>
       <geometry>
-        <box size=".4 .2 .1"/>
+        <box size=".6 .4 .1"/>
       </geometry>
     </collision>
@@ -28,5 +28,5 @@
       <origin xyz="0 0 0" rpy=" 0 0 0"/>
       <geometry>
-        <box size=".4 .2 .1"/>
+        <box size=".6 .4 .1"/>
       </geometry>
          <material name="green"/>
@@ -70,5 +70,5 @@
       <origin xyz="0 0 0" rpy=" 0 1.5707 1.5707"/>
       <geometry>
-        <cylinder radius="0.1" length="0.05"/>
+        <cylinder radius="0.09" length="0.03"/>
       </geometry>
     </collision>
@@ -76,5 +76,5 @@
       <origin xyz="0 0 0" rpy=" 0 1.5707 1.5707"/>
       <geometry>
-        <cylinder radius="0.1" length="0.05"/>
+        <cylinder radius="0.09" length="0.03"/>
       </geometry>
          <material name="green"/>
@@ -82,5 +82,5 @@
 </link>
 <joint type="continuous" name="left_wheel_hinge">
-    <origin xyz="0 0.15 0" rpy="0 0 0"/>
+    <origin xyz="0 0.23 0" rpy="0 0 0"/>
     <child link="LEFT_wheel"/>
     <parent link="chassis"/>
@@ -102,5 +102,5 @@
       <origin xyz="0 0 0" rpy=" 0 1.5707 1.5707"/>
       <geometry>
-        <cylinder radius="0.1" length="0.05"/>
+        <cylinder radius="0.09" length="0.03"/>
       </geometry>
     </collision>
@@ -108,5 +108,5 @@
       <origin xyz="0 0 0" rpy=" 0 1.5707 1.5707"/>
       <geometry>
-        <cylinder radius="0.1" length="0.05"/>
+        <cylinder radius="0.09" length="0.03"/>
       </geometry>
          <material name="green"/>
@@ -114,5 +114,5 @@
 </link>
 <joint type="continuous" name="right_wheel_hinge">
-    <origin xyz="0 -0.15 0" rpy="0 0 0"/>
+    <origin xyz="0 -0.23 0" rpy="0 0 0"/>
     <child link="RIGHT_wheel"/>
     <parent link="chassis"/>
@@ -146,5 +146,5 @@
 </link>
 <joint type="fixed" name="camera_joint">
-    <origin xyz="0.2 0 0" rpy="0 0 0"/>
+    <origin xyz="0.3 0 0" rpy="0 0 0"/>
     <child link="camera"/>
     <parent link="chassis"/>

Commit message: Updated robot to have a cylinder body and moved color to xacro file

File: catkin_ws/src/my_robot/urdf/my_robot.xacro (robot description, xacro)
@@ -22,5 +22,5 @@
       <origin xyz="0 0 0" rpy=" 0 0 0"/>
       <geometry>
-        <box size=".6 .4 .1"/>
+        <cylinder radius="0.2" length="0.1"/>
       </geometry>
     </collision>
@@ -28,10 +28,10 @@
       <origin xyz="0 0 0" rpy=" 0 0 0"/>
       <geometry>
-        <box size=".6 .4 .1"/>
+        <cylinder radius="0.2" length="0.1"/>
       </geometry>
          <material name="green"/>
     </visual>
     <collision name='back_caster_collision'>
-      <origin xyz="-0.15 0 -0.05" rpy=" 0 0 0"/>
+      <origin xyz="-0.1 0 -0.05" rpy=" 0 0 0"/>
       <geometry>
         <sphere radius="0.0499"/>
@@ -39,5 +39,5 @@
     </collision>
     <visual name='back_caster_visual'>
-      <origin xyz="-0.15 0 -0.05" rpy=" 0 0 0"/>
+      <origin xyz="-0.1 0 -0.05" rpy=" 0 0 0"/>
       <geometry>
         <sphere radius="0.05"/>
@@ -45,5 +45,5 @@
     </visual>
     <collision name='front_caster_collision'>
-      <origin xyz="0.15 0 -0.05" rpy=" 0 0 0"/>
+      <origin xyz="0.1 0 -0.05" rpy=" 0 0 0"/>
       <geometry>
         <sphere radius="0.0499"/>
@@ -51,5 +51,5 @@
     </collision>
     <visual name='front_caster_visual'>
-      <origin xyz="0.15 0 -0.05" rpy=" 0 0 0"/>
+      <origin xyz="0.1 0 -0.05" rpy=" 0 0 0"/>
       <geometry>
         <sphere radius="0.05"/>
@@ -146,5 +146,5 @@
 </link>
 <joint type="fixed" name="camera_joint">
-    <origin xyz="0.3 0 0" rpy="0 0 0"/>
+    <origin xyz="0.20 0 0" rpy="0 0 0"/>
     <child link="camera"/>
     <parent link="chassis"/>
@@ -175,8 +175,14 @@
 </link>
 <joint type="fixed" name="hokuyo_joint">
-    <origin xyz="0.15 0 .1" rpy="0 0 0"/>
+    <origin xyz="0.125 0 .1" rpy="0 0 0"/>
     <child link="hokuyo"/>
     <parent link="chassis"/>
     <axis xyz="0 1 0" rpy="0 0 0"/>
 </joint>
+<gazebo reference="LEFT_wheel">
+    <material>Gazebo/Yellow</material>
+</gazebo>
+<gazebo reference="RIGHT_wheel">
+    <material>Gazebo/Yellow</material>
+</gazebo>
 </robot>

Commit message: Enhanced following white ball; fixed duplicate model in world file

File: catkin_ws/src/my_robot/urdf/my_robot.xacro (robot description, xacro)
@@ -70,5 +70,5 @@
       <origin xyz="0 0 0" rpy=" 0 1.5707 1.5707"/>
       <geometry>
-        <cylinder radius="0.09" length="0.03"/>
+        <cylinder radius="0.1" length="0.03"/>
       </geometry>
     </collision>
@@ -76,5 +76,5 @@
       <origin xyz="0 0 0" rpy=" 0 1.5707 1.5707"/>
       <geometry>
-        <cylinder radius="0.09" length="0.03"/>
+        <cylinder radius="0.1" length="0.03"/>
       </geometry>
          <material name="green"/>
@@ -102,5 +102,5 @@
       <origin xyz="0 0 0" rpy=" 0 1.5707 1.5707"/>
       <geometry>
-        <cylinder radius="0.09" length="0.03"/>
+        <cylinder radius="0.1" length="0.03"/>
       </geometry>
     </collision>
@@ -108,5 +108,5 @@
       <origin xyz="0 0 0" rpy=" 0 1.5707 1.5707"/>
       <geometry>
-        <cylinder radius="0.09" length="0.03"/>
+        <cylinder radius="0.1" length="0.03"/>
       </geometry>
          <material name="green"/>
